File: Solfacon.kicad_pcb (KiCad board)
At the start: 2 copper layers, 48 x 73 mm, 50 parts, among them Q1 TSM480P06, Q2 TP0606, Q3 ZVN3306A, Q4 STP55NF06L, U1 ATtiny85

Commit message: Add files via upload
Parts:
- D5: value 1N5817 -> SB140
- R1, R5: value 47K -> 22K
- R3: value 330 -> 200
- moved C12 0.20 mm to (65.4, 46.5)

Commit message: Readme updated
Parts:
- C7, C8: value 0.6F -> 1F
Changed lines of the file:
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@@
     (descr "SCMR14L334SSBB0-1")
     (tags "Capacitor Polarised")
-    (property "Arrow Part Number" "SCMR14L334SSBB0")
-    (property "Arrow Price/Stock" "https://www.arrow.com/en/products/scmr14l334ssbb0/avx")
-    (property "Datasheet_1" "https://datasheets.kyocera-avx.com/AVX-SCM.pdf")
-    (property "Footprint_1" "SCMR14L334SSBB0")
-    (property "Height" "18")
-    (property "Manufacturer_Name" "Kyocera AVX")
-    (property "Manufacturer_Part_Number" "SCMR14L334SSBB0")
-    (property "Mouser Part Number" "581-SCMR14L334SSBB0")
-    (property "Mouser Price/Stock" "https://www.mouser.com/Search/Refine.aspx?Keyword=581-SCMR14L334SSBB0")
     (property "Reference_1" "C")
     (property "Sheetfile" "Solfacon.kicad_sch")
     (property "Sheetname" "")
-    (property "Value_1" "SCMR14L334SSBB0")
     (attr through_hole)
     (fp_text reference "C8" (at 6.75 0) (layer "F.SilkS")
       (effects (font (size 0.9 0.9) (thickness 0.15)))
     )
-    (fp_text value "0.6F" (at 6.75 0) (layer "F.SilkS") hide
+    (fp_text value "1F" (at 6.75 0) (layer "F.SilkS") hide
       (effects (font (size 1.27 1.27) (thickness 0.254)))
     )
@@
     (descr "SCMR14L334SSBB0-1")
     (tags "Capacitor Polarised")
-    (property "Arrow Part Number" "SCMR14L334SSBB0")
-    (property "Arrow Price/Stock" "https://www.arrow.com/en/products/scmr14l334ssbb0/avx")
-    (property "Datasheet_1" "https://datasheets.kyocera-avx.com/AVX-SCM.pdf")
-    (property "Footprint_1" "SCMR14L334SSBB0")
-    (property "Height" "18")
-    (property "Manufacturer_Name" "Kyocera AVX")
-    (property "Manufacturer_Part_Number" "SCMR14L334SSBB0")
-    (property "Mouser Part Number" "581-SCMR14L334SSBB0")
-    (property "Mouser Price/Stock" "https://www.mouser.com/Search/Refine.aspx?Keyword=581-SCMR14L334SSBB0")
     (property "Reference_1" "C")
     (property "Sheetfile" "Solfacon.kicad_sch")
     (property "Sheetname" "")
-    (property "Value_1" "SCMR14L334SSBB0")
     (attr through_hole)
     (fp_text reference "C7" (at 6.75 0) (layer "F.SilkS")
       (effects (font (size 0.9 0.9) (thickness 0.15)))
     )
-    (fp_text value "0.6F" (at 6.75 0) (layer "F.SilkS") hide
+    (fp_text value "1F" (at 6.75 0) (layer "F.SilkS") hide
       (effects (font (size 1.27 1.27) (thickness 0.254)))
     )
@@
   (dimension (type aligned) (layer "Cmts.User")
     (pts (xy 73.988286 91.640131) (xy 33.988286 91.640131))
-    (height -19.5)
-    (gr_text "40,0000 mm" (at 53.988286 110.090131) (layer "Cmts.User")
+    (height -15.359869)
+    (gr_text "40,0000 mm" (at 53.988286 105.95) (layer "Cmts.User")
       (effects (font (size 0.9 0.9) (thickness 0.15)))
     )
     (format (units 3) (units_format 1) (precision 4))
-    (style (thickness 0.12) (arrow_length 1.27) (text_position_mode 0) (extension_height 0.58642) (extension_offset 0.5) keep_text_aligned)
+    (style (thickness 0.1) (arrow_length 1.27) (text_position_mode 0) (extension_height 0.58642) (extension_offset 0.5) keep_text_aligned)
   )
   (dimension (type aligned) (layer "Cmts.User")
     (pts (xy 53.988286 50.343936) (xy 53.988286 58.143936))
     (height 29)
-    (gr_text "7,8000 mm" (at 23.838286 54.243936 90) (layer "Cmts.User")
-      (effects (font (size 1 1) (thickness 0.15)))
+    (gr_text "7,8000 mm" (at 23.938286 54.243936 90) (layer "Cmts.User")
+      (effects (font (size 0.9 0.9) (thickness 0.15)))
     )
     (format (units 3) (units_format 1) (precision 4))
@@
   (dimension (type aligned) (layer "Cmts.User")
     (pts (xy 73.988286 41.640131) (xy 73.988286 91.640131))
-    (height -16)
-    (gr_text "50,0000 mm" (at 88.938286 66.640131 90) (layer "Cmts.User")
+    (height -9.011714)
+    (gr_text "50,0000 mm" (at 81.95 66.640131 90) (layer "Cmts.User")
       (effects (font (size 0.9 0.9) (thickness 0.15)))
     )
     (format (units 3) (units_format 1) (precision 4))
-    (style (thickness 0.12) (arrow_length 1.27) (text_position_mode 0) (extension_height 0.58642) (extension_offset 0.5) keep_text_aligned)
+    (style (thickness 0.1) (arrow_length 1.27) (text_position_mode 0) (extension_height 0.58642) (extension_offset 0.5) keep_text_aligned)
   )
   (segment (start 42 52.087449) (end 41.535666 52.087449) (width 0.6) (layer "F.Cu") (net 2))
