File: Solfacon.kicad_sch (KiCad schematic)
At the start: 39 parts, among them Q1 TSM480P06, Q2 TP0606, Q3 ZVN3306A, Q4 STP55NF06L, U1 ATtiny85

Commit message: Add files via upload
Parts:
- R5: value 47K -> 22K
Changed lines of the file:
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@@
       (effects (font (size 1.27 1.27)) (justify left))
     )
-    (property "Value" "47K" (id 1) (at 252.73 124.4599 0)
+    (property "Value" "22K" (id 1) (at 252.73 124.4599 0)
       (effects (font (size 1.27 1.27)) (justify left))
     )
@@
     )
     (path "/893417e2-af74-42ca-9d57-82d50ee39e4d"
-      (reference "R5") (unit 1) (value "47K") (footprint "Resistor_THT:R_Axial_DIN0207_L6.3mm_D2.5mm_P2.54mm_Vertical")
+      (reference "R5") (unit 1) (value "22K") (footprint "Resistor_THT:R_Axial_DIN0207_L6.3mm_D2.5mm_P2.54mm_Vertical")
     )
     (path "/c4f02467-017f-4944-972b-46b24ad8770a"

Commit message: Readme updated
Parts:
- C7, C8: value 0.6F -> 1F; Arrow Part Number SCMR14L334SSBB0 -> (none); Arrow Price/Stock https://www.arrow.com/en/products/scmr14l334ssbb0/avx -> (none); Datasheet_1 https://datasheets.kyocera-avx.com/AVX-SCM.pdf -> (none); Footprint_1 SCMR14L334SSBB0 -> (none); Height 18 -> (none); Manufacturer_Name Kyocera AVX -> (none); Manufacturer_Part_Number SCMR14L334SSBB0 -> (none); Mouser Part Number 581-SCMR14L334SSBB0 -> (none); Mouser Price/Stock https://www.mouser.com/Search/Refine.aspx?Keyword=581-SCMR1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 -> (none); Value_1 SCMR14L334SSBB0 -> (none)
Changed lines of the file:
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@@
       (effects (font (size 1.27 1.27)) (justify left))
     )
-    (property "Value" "0.6F" (id 1) (at 190.5 54.61 90)
+    (property "Value" "1F" (id 1) (at 190.5 54.61 90)
       (effects (font (size 1.27 1.27)) (justify left))
     )
@@
     (property "Reference_1" "C" (id 4) (at 194.31 53.34 0)
       (effects (font (size 1.27 1.27)) hide)
-    )
-    (property "Value_1" "SCMR14L334SSBB0" (id 5) (at 191.77 53.34 0)
-      (effects (font (size 1.27 1.27)) hide)
-    )
-    (property "Footprint_1" "SCMR14L334SSBB0" (id 6) (at 90.5 50.8 0)
-      (effects (font (size 1.27 1.27)) (justify left top) hide)
-    )
-    (property "Datasheet_1" "https://datasheets.kyocera-avx.com/AVX-SCM.pdf" (id 7) (at -9.5 50.8 0)
-      (effects (font (size 1.27 1.27)) (justify left top) hide)
-    )
-    (property "Height" "18" (id 8) (at -209.5 50.8 0)
-      (effects (font (size 1.27 1.27)) (justify left top) hide)
-    )
-    (property "Manufacturer_Name" "Kyocera AVX" (id 9) (at -309.5 50.8 0)
-      (effects (font (size 1.27 1.27)) (justify left top) hide)
-    )
-    (property "Manufacturer_Part_Number" "SCMR14L334SSBB0" (id 10) (at -409.5 50.8 0)
-      (effects (font (size 1.27 1.27)) (justify left top) hide)
-    )
-    (property "Mouser Part Number" "581-SCMR14L334SSBB0" (id 11) (at -509.5 50.8 0)
-      (effects (font (size 1.27 1.27)) (justify left top) hide)
-    )
-    (property "Mouser Price/Stock" "https://www.mouser.com/Search/Refine.aspx?Keyword=581-SCMR14L334SSBB0" (id 12) (at -609.5 50.8 0)
-      (effects (font (size 1.27 1.27)) (justify left top) hide)
-    )
-    (property "Arrow Part Number" "SCMR14L334SSBB0" (id 13) (at -709.5 50.8 0)
-      (effects (font (size 1.27 1.27)) (justify left top) hide)
-    )
-    (property "Arrow Price/Stock" "https://www.arrow.com/en/products/scmr14l334ssbb0/avx" (id 14) (at -809.5 50.8 0)
-      (effects (font (size 1.27 1.27)) (justify left top) hide)
     )
     (pin "1")
@@
     (in_bom yes) (on_board yes)
     (property "Reference" "C8" (id 0) (at 191.77 38.1 90))
-    (property "Value" "0.6F" (id 1) (at 190.5 40.64 90)
+    (property "Value" "1F" (id 1) (at 190.5 40.64 90)
       (effects (font (size 1.27 1.27)) (justify left))
     )
@@
     (property "Reference_1" "C" (id 4) (at 194.31 39.37 0)
       (effects (font (size 1.27 1.27)) hide)
-    )
-    (property "Value_1" "SCMR14L334SSBB0" (id 5) (at 191.77 39.37 0)
-      (effects (font (size 1.27 1.27)) hide)
-    )
-    (property "Footprint_1" "SCMR14L334SSBB0" (id 6) (at 90.5 36.83 0)
-      (effects (font (size 1.27 1.27)) (justify left top) hide)
-    )
-    (property "Datasheet_1" "https://datasheets.kyocera-avx.com/AVX-SCM.pdf" (id 7) (at -9.5 36.83 0)
-      (effects (font (size 1.27 1.27)) (justify left top) hide)
-    )
-    (property "Height" "18" (id 8) (at -209.5 36.83 0)
-      (effects (font (size 1.27 1.27)) (justify left top) hide)
-    )
-    (property "Manufacturer_Name" "Kyocera AVX" (id 9) (at -309.5 36.83 0)
-      (effects (font (size 1.27 1.27)) (justify left top) hide)
-    )
-    (property "Manufacturer_Part_Number" "SCMR14L334SSBB0" (id 10) (at -409.5 36.83 0)
-      (effects (font (size 1.27 1.27)) (justify left top) hide)
-    )
-    (property "Mouser Part Number" "581-SCMR14L334SSBB0" (id 11) (at -509.5 36.83 0)
-      (effects (font (size 1.27 1.27)) (justify left top) hide)
-    )
-    (property "Mouser Price/Stock" "https://www.mouser.com/Search/Refine.aspx?Keyword=581-SCMR14L334SSBB0" (id 12) (at -609.5 36.83 0)
-      (effects (font (size 1.27 1.27)) (justify left top) hide)
-    )
-    (property "Arrow Part Number" "SCMR14L334SSBB0" (id 13) (at -709.5 36.83 0)
-      (effects (font (size 1.27 1.27)) (justify left top) hide)
-    )
-    (property "Arrow Price/Stock" "https://www.arrow.com/en/products/scmr14l334ssbb0/avx" (id 14) (at -809.5 36.83 0)
-      (effects (font (size 1.27 1.27)) (justify left top) hide)
     )
     (pin "1")
@@
     )
     (path "/62640d88-0e67-4db7-8229-c21e40fa81c5"
-      (reference "C7") (unit 1) (value "0.6F") (footprint "components:SCMR14L334SSBB0")
+      (reference "C7") (unit 1) (value "1F") (footprint "components:SCMR14L334SSBB0")
     )
     (path "/c8975573-1a88-4a63-a257-5fd20f551dd4"
-      (reference "C8") (unit 1) (value "0.6F") (footprint "components:SCMR14L334SSBB0")
+      (reference "C8") (unit 1) (value "1F") (footprint "components:SCMR14L334SSBB0")
     )
     (path "/ddd95d88-ec0d-4e14-b28c-3540703d14d9"
